File: pcb/main.kicad_pcb (KiCad board)
At the start: 2 copper layers, 292.6 x 146.9 mm, 143 parts, among them J1 https://datasheet.lcsc.com/lc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, SW1 SW_Push, SW10 SW_Push, SW11 SW_Push, SW12 SW_Push, SW13 SW_Push, SW14 SW_Push, SW15 SW_Push, SW16 SW_Push, SW17 SW_Push, SW18 SW_Push, SW19 SW_Push, SW2 SW_Push, SW20 SW_Push, SW21 SW_Push, SW22 SW_Push, SW23 SW_Push, SW24 SW_Push, SW25 SW_Push, SW26 SW_Push, SW27 SW_Push, SW28 SW_Push, SW29 SW_Push, SW3 SW_Push, SW30 SW_Push, SW31 SW_Push, SW32 SW_Push, SW33 SW_Push, SW34 SW_Push, SW35 SW_Push, SW36 SW_Push, SW37 SW_Push, SW38 SW_Push, SW39 SW_Push, SW4 SW_Push, SW40 SW_Push, SW41 SW_Push, SW42 SW_Push, SW43 SW_Push, SW44 SW_Push, SW45 SW_Push, SW46 SW_Push, SW47 SW_Push, SW48 SW_Push, SW49 SW_Push, SW5 SW_Push, SW50 SW_Push, SW51 SW_Push, SW52 SW_Push, SW53 SW_Push, SW54 SW_Push, SW55 SW_Push, SW56 SW_Push, SW57 SW_Push, SW58 SW_Push, SW59 SW_Push, SW6 SW_Push, SW60 SW_Push, SW61 RST, SW62 RST, SW7 SW_Push, SW8 SW_Push, SW9 SW_Push, U1 USBLC6-2SC6, U2 AP2204R-3.3, U3 STM32L072KZTx

Commit message: Fixed missing columns, fixed USB-C connector position, new LDO
Parts:
- U2: value AP2204R-3.3 -> HT75xx-1-SOT89
- moved C2 6.25 mm to (-192.8, 57.8)
- moved C1 1.90 mm to (-192.8, 50.2)
- moved J1 1.39 mm to (-198.4, 30.9)
- moved U2 1.25 mm to (-192.0, 54.0), turned to 0 degrees
- moved R5 1.06 mm to (-198.0, 70.2), turned to 0 degrees
- moved D42 0.67 mm to (-165.5, 82.5)
- turned SW57 to -117.5 degrees
Connections:
- D18 pad 1: /keys/col5 -> /MCU/A1
- D19 pad 1: /keys/col6 -> /MCU/A0
- D30 pad 1: /keys/col5 -> /MCU/A1
- D31 pad 1: /keys/col6 -> /MCU/A0
- D42 pad 1: /keys/col5 -> /MCU/A1
- D43 pad 1: /keys/col6 -> /MCU/A0
- D54 pad 1: /keys/col5 -> /MCU/A1
- D55 pad 1: /keys/col6 -> /MCU/A0
- D6 pad 1: /keys/col5 -> /MCU/A1
- D7 pad 1: /keys/col6 -> /MCU/A0
- U2 pad 1: VBUS -> GND
- U2 pad 2: GND -> VBUS
Routing:
- net /MCU/A0: track 0.00 -> 111.4 mm
- net /MCU/A1: track 0.00 -> 97.5 mm
- net /keys/col6: track 58.0 -> 0.00 mm
- net /keys/col5: track 58.0 -> 0.00 mm
- net /MCU/A2: track 306.0 -> 329.1 mm
- net Net-(D57-Pad2): track 17.6 -> 7.50 mm
- net /MCU/A3: track 165.8 -> 172.5 mm
- net GND: track 38.3 -> 33.3 mm, vias 6 -> 7
- net /MCU/B6: track 164.2 -> 161.2 mm
- net /MCU/B7: track 342.3 -> 339.5 mm
- net /MCU/C15: track 288.6 -> 287.2 mm
- net /MCU/C14: track 320.2 -> 319.2 mm
- net /MCU/A5: track 178.5 -> 177.7 mm
- net /MCU/B0: track 240.1 -> 239.3 mm
