File: pcb/main.kicad_sch (KiCad schematic)
At the start: 16 parts, among them J1 https://datasheet.lcsc.com/lc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, SW61 RST, SW62 RST, U1 USBLC6-2SC6

Commit message: Fixed missing columns, fixed USB-C connector position, new LDO
Connections:
- no-connect marks 2 -> 8
Other:
- sheet MCU ports: added A1, A10, A13, A14, A9, B1; removed none
Changed lines of the file:
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@@
   (junction (at 91.44 74.93) (diameter 0) (color 0 0 0 0)
   )
+  (no_connect (at 161.29 129.54))
+  (no_connect (at 161.29 132.08))
+  (no_connect (at 161.29 134.62))
+  (no_connect (at 161.29 137.16))
+  (no_connect (at 161.29 139.7))
+  (no_connect (at 161.29 142.24))
   (no_connect (at 106.68 67.31))
   (no_connect (at 106.68 64.77))
@@
     (stroke (width 0) (type default) (color 0 0 0 0))
   )
+  (wire (pts (xy 194.31 124.46) (xy 210.82 124.46))
+    (stroke (width 0) (type default) (color 0 0 0 0))
+  )
   (wire (pts (xy 194.31 106.68) (xy 210.82 106.68))
     (stroke (width 0) (type default) (color 0 0 0 0))
@@
   )
   (wire (pts (xy 130.81 49.53) (xy 130.81 43.18))
+    (stroke (width 0) (type default) (color 0 0 0 0))
+  )
+  (wire (pts (xy 194.31 142.24) (xy 210.82 142.24))
     (stroke (width 0) (type default) (color 0 0 0 0))
   )
@@
     (effects (font (size 1.27 1.27)) (justify right bottom))
   )
-  (global_label "VBUS" (shape input) (at 106.68 36.83 0) (fields_autoplaced)
+  (global_label "VBUS" (shape output) (at 106.68 36.83 0) (fields_autoplaced)
     (effects (font (size 1.27 1.27)) (justify left))
-    (property "Intersheet References" "${INTERSHEET_REFS}" (id 0) (at 55.88 13.97 0)
-      (effects (font (size 1.27 1.27)) hide)
+    (property "Intersheet References" "${INTERSHEET_REFS}" (id 0) (at 113.9028 36.7506 0)
+      (effects (font (size 1.27 1.27)) (justify left) hide)
     )
   )
@@
       (effects (font (size 1.27 1.27)) (justify right))
     )
-    (pin "A8" bidirectional (at 185.42 92.71 90)
-      (effects (font (size 1.27 1.27)) (justify right))
-    )
     (pin "A4" bidirectional (at 194.31 96.52 0)
       (effects (font (size 1.27 1.27)) (justify right))
@@
     (pin "A3" bidirectional (at 194.31 139.7 0)
       (effects (font (size 1.27 1.27)) (justify right))
+    )
+    (pin "A1" bidirectional (at 194.31 142.24 0)
+      (effects (font (size 1.27 1.27)) (justify right))
+    )
+    (pin "B1" bidirectional (at 161.29 142.24 180)
+      (effects (font (size 1.27 1.27)) (justify left))
+    )
+    (pin "A9" bidirectional (at 161.29 132.08 180)
+      (effects (font (size 1.27 1.27)) (justify left))
+    )
+    (pin "A8" bidirectional (at 161.29 129.54 180)
+      (effects (font (size 1.27 1.27)) (justify left))
+    )
+    (pin "A10" bidirectional (at 161.29 134.62 180)
+      (effects (font (size 1.27 1.27)) (justify left))
+    )
+    (pin "A13" bidirectional (at 161.29 137.16 180)
+      (effects (font (size 1.27 1.27)) (justify left))
+    )
+    (pin "A14" bidirectional (at 161.29 139.7 180)
+      (effects (font (size 1.27 1.27)) (justify left))
     )
   )
@@
       (reference "U1") (unit 1) (value "USBLC6-2SC6") (footprint "Package_TO_SOT_SMD:SOT-23-6")
     )
-    (path "/bc3548e8-a5f2-4ff9-a75d-79736bf75a82/74dfd341-0a7b-485e-bf92-711dd2c4ba6f"
-      (reference "U2") (unit 1) (value "AP2204R-3.3") (footprint "Package_TO_SOT_SMD:SOT-89-3")
+    (path "/bc3548e8-a5f2-4ff9-a75d-79736bf75a82/312dda7e-4990-416b-8d34-829a226c1479"
+      (reference "U2") (unit 1) (value "HT75xx-1-SOT89") (footprint "Package_TO_SOT_SMD:SOT-89-3")
     )
     (path "/bc3548e8-a5f2-4ff9-a75d-79736bf75a82/151a21a1-d307-4f78-82dc-6f5f0b9459ea"
