File: pcb/mcu.kicad_sch (KiCad schematic)
At the start: 7 parts, among them U2 AP2204R-3.3, U3 STM32L072KZTx

Commit message: Fixed missing columns, fixed USB-C connector position, new LDO
Parts:
- removed U2: AP2204R-3.3, Package_TO_SOT_SMD:SOT-89-3, symbol Regulator_Linear:AP2204R-3.3
- added U2: HT75xx-1-SOT89, Package_TO_SOT_SMD:SOT-89-3, symbol Regulator_Linear:HT75xx-1-SOT89
Connections:
- net GND: now also U2.1 (GND)
- net VBUS: now also U2.2 (VIN)
- net VSTM: now also U2.3 (VOUT)
Changed lines of the file:
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@@
     (pin "9")
+  )
+  (symbol (lib_id "Regulator_Linear:HT75xx-1-SOT89") (at 62.23 53.34 0) (unit 1)
+    (in_bom yes) (on_board yes) (fields_autoplaced)
+    (property "Reference" "U2" (id 0) (at 62.23 44.2935 0))
+    (property "Value" "HT75xx-1-SOT89" (id 1) (at 62.23 47.0686 0))
+    (property "Footprint" "Package_TO_SOT_SMD:SOT-89-3" (id 2) (at 62.23 45.085 0)
+      (effects (font (size 1.27 1.27) italic) hide)
+    )
+    (property "Datasheet" "https://www.holtek.com/documents/10179/116711/HT75xx-1v250.pdf" (id 3) (at 62.23 50.8 0)
+      (effects (font (size 1.27 1.27)) hide)
+    )
+    (property "LCSC" "C14289" (id 4) (at 62.23 53.34 0)
+      (effects (font (size 1.27 1.27)) hide)
+    )
+    (pin "1")
+    (pin "2")
+    (pin "3")
   )
   (symbol (lib_id "power:GND") (at 102.87 59.69 0) (unit 1)
@@
     (pin "2")
   )
-  (symbol (lib_id "Regulator_Linear:AP2204R-3.3") (at 62.23 50.8 0) (unit 1)
-    (in_bom yes) (on_board yes) (fields_autoplaced)
-    (property "Reference" "U2" (id 0) (at 62.23 44.9285 0))
-    (property "Value" "AP2204R-3.3" (id 1) (at 62.23 47.7036 0))
-    (property "Footprint" "Package_TO_SOT_SMD:SOT-89-3" (id 2) (at 62.23 45.085 0)
-      (effects (font (size 1.27 1.27)) hide)
-    )
-    (property "Datasheet" "https://www.diodes.com/assets/Datasheets/AP2204.pdf" (id 3) (at 62.23 50.8 0)
-      (effects (font (size 1.27 1.27)) hide)
-    )
-    (pin "1")
-    (pin "2")
-    (pin "3")
-  )
   (symbol (lib_id "Device:R") (at 90.17 82.55 180) (unit 1)
